File: PCB/ShutterControl/ShutterControl.kicad_sch (KiCad schematic)
At the start: 13 parts, among them J1 Battery +, J2 Battery -, SW1 Button1, SW2 Button2, SW3 Button3, SW4 Button4, U1 ESP32-C3_SUPERMINI_TH

Commit message: Solved an error with committing
Parts:
- removed R4: 10k, Resistor_THT:R_Axial_DIN0204_L3.6mm_D1.6mm_P5.08mm_Horizontal, symbol Device:R
- removed SW4: Button4, Button_Switch_THT:SW_PUSH_6mm_H5mm, symbol Switch:SW_Push
- SW1: value Button1 -> UP
- SW2: value Button2 -> STOP
- SW3: value Button3 -> DOWN
Connections:
- net at U1.4 (GPIO4): now also R2.2, SW2.2
- now unconnected: U1.2 (GPIO2)
